Commit message: feat(scene): rotating pulleys, holder rim collision, belt on the rim, 2F-85 seat
- Task-board pulleys are unactuated revolute joints (URDF continuous, damping
  0.001) solved with the belt in the VBD entry; the loader turns root-parented
  revolute links into bodies and filters their collisions with the board.
- Belt holder gains collision quarters for its slotted outer rim; the belt is
  resized to rest on the rim against the middle-tier wall, with the stretch
  stiffness from the MISUMI MBT6-640 datasheet (16.6 N at 5%).
- The 2F-85 sits 3 mm into the UR10 flange (the coupling's pocket), putting
  the fingertips at 194 mm, as magna's finger_tip_frame.
- Vendors dairlib lcmt_object_state; adds check_pulleys and extends the
  directive, pose and lcmtypes checks.

File: assets/common/belt_chain_holder/belt_chain_holder.urdf (robot description, URDF)
Before this commit: robot belt_chain_holder, 2 links, 1 joints
Links:
- link belt_chain_holder_first_half: geometry collision mesh filename=bottom_plate.obj; collision mesh filename=quarter_ellipse_bottom.obj
- link belt_chain_holder_second_half: geometry collision mesh filename=quarter_ellipse_bottom.obj; collision mesh filename=quarter_ellipse_bottom.obj

File: assets/round_belt_task/round_belt_task_board.urdf (robot description, URDF)
Before this commit: robot task_board, 3 links, 2 joints
Links:
- link large_round_pulley: geometry collision mesh filename=round_belt_task_board/large_round_pulley/large_round_pulley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 scale=0.001 0.001 0.001; collision mesh filename=round_belt_task_board/large_round_pulley/large_round_pulley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 scale=0.001 0.001 0.001
- link small_round_pulley: geometry collision mesh filename=round_belt_task_board/small_round_pulley/small_round_pulley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 scale=0.001 0.001 0.001; collision mesh filename=round_belt_task_board/small_round_pulley/small_round_pulley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 scale=0.001 0.001 0.001
Joints:
- joint large_round_pulley_joint: axis (none) -> 0 0 1; limit (none) -> effort=0 velocity=100; origin xyz=0 0 0 rpy=0 0 0 -> xyz=0.140 0.196 0.0248 rpy=0 0 0; type fixed -> continuous
- joint small_round_pulley_joint: axis (none) -> 0 0 1; limit (none) -> effort=0 velocity=100; origin xyz=0 0 0 rpy=0 0 0 -> xyz=0.355 0.196 0.0248 rpy=0 0 0; type fixed -> continuous
